File: High Temp Load Cell Toolhead Board/High Temp Load Cell Toolhead Board.kicad_sch (KiCad schematic)
At the start: 110 parts, among them J1 Conn_01x03, J11 Conn_01x03, J12 Conn_01x03, J13 PinHeader_2x4_P2.54mm, J2 Conn_02x08, J6 Conn_01x04, J7 Conn_01x02, J8 Conn_01x04, J9 Conn_01x02, Q1 DMG3404L, Q2 DMG3404L, SW1 SW_SPST, U1 MAX31865xTP, U2 STM32F103CBU6TR, U3 SN74LVC2G17DSFR, U4 SN74AHC1G32QDBVRQ1, U5 ADS1220, X1 ECS-2520MVLC-080-BP-TR

Commit message: Add USB C Connector
The commit adds a USB C connector to the back side of the board.
* This can be used to bench run and test the board without the 24V power supply.
* Its not designed to be used with the printer is operational, thats what the main connector is for
* All components are optional and can be omitted
* Reverse current protection diodes are included to stop current backfeeding into the USB Host in operation

Other updates:
* Add 3D Models for the VRM components
* ADS1220 clock pin should have been tied to ground
* ADS1220 pad 17 can be connected to AVSS, which is GND in this design
* Add QR Code with URL to the project, name and version to the back side
* Add 3 fiducial markers in case someone wants to run this on a pick and place machine
Parts:
- added D15, D16: 40V, 1A, SMA, Diode_SMD:D_SMA, symbol Device:D_Schottky
- added FID1, FID2, FID3: Fiducial, Fiducial:Fiducial_0.5mm_Mask1.5mm, symbol Mechanical:Fiducial
- added P1: USB_C_Plug_USB2.0, Connector_USB:USB_C_Receptacle_GCT_USB4110, symbol Connector:USB_C_Receptacle_USB2.0_16P
- added R6, R7: R5.1kΩ, Resistor_SMD:R_0603_1608Metric, symbol Device:R
- D3: now fitted
- LDO1: Supplier_Link https://www.mouser.com/ProductDetail/Texas-Instruments/TPS7A2150PQWDRBRQ1 -> https://www.mouser.com/ProductDetail/Texas-Instruments/TPS7A2150PQWDRBRQ1?qs=ZcfC38r4PotpxWDbDIZdAw%3D%3D
Connections:
- net +5V: now also D16.1 (K)
- net +5V5: now also D15.1 (K)
- net GND: now also U5.17 (THERMAL), U5.3 (CLK), P1.A1 (GND), P1.A12 (GND), P1.B1 (GND), P1.B12 (GND), R6.2, R7.2
- net USB_D+: now also P1.A6 (D+), P1.B6 (D+)
- net USB_D-: now also P1.A7 (D-), P1.B7 (D-)
- new net: P1.A5 (CC1), R6.1
- new net: P1.B5 (CC2), R7.1
- new net: D15.2 (A), D16.2 (A), P1.A4 (VBUS), P1.A9 (VBUS), P1.B4 (VBUS), P1.B9 (VBUS)
- no-connect marks 25 -> 28
Other:
- note added: "USBC Connector (Optional)"
- moved on the sheet: C31, J13, R27

Commit message: Add Net Class Directives
This change adds Net Class Directives for 3 types of specialized nets:
* ADC Signal - a net that may potentially be sensed by an ADC and should be treated as 50 Ohm impedance
* Digital Signal - a net that will have an oscillating digital signal on it but does not carry any power. This should also be treated as 50 Ohm impedance.
* Digital Pair - a differential digital pair. This is only used for the USB data pair which is 90 Ohm impedance.
Connections:
- net INPUT_24V+ renamed +24V_INPUT
- net INPUT_FANV+ renamed +FANV_INPUT
- net SPI_2_SCLK renamed LED_MCU_CLK
- net SPI_2_SDO renamed LED_MCU_SDO
- no-connect marks 28 -> 27
Other:
- moved on the sheet: C12, C13, C14, C15, C16, D4, L4, L5, R16, R17, U5
